Commit message: Fix relative urdf positioning.

File: src/util/twoTwoBarDiffLength.urdf (robot description, URDF)
Before this commit: robot DoublePendulum, 5 links, 4 joints
Joints:
- joint joint1: origin xyz=0 0 0 -> xyz=0 0 0 rpy=0. 0 0
- joint joint2: origin xyz=0 0 -1 -> xyz=0 0 -1 rpy=-0.2 0 0
- joint joint3: origin xyz=0 0 0 -> xyz=0 1 0 rpy=0.5 0 0

Commit message: Save current state.

File: src/util/twoTwoBarDiffLength.urdf (robot description, URDF)
Before this commit: robot DoublePendulum, 5 links, 4 joints
Joints:
- joint joint1: origin xyz=0 0 0 rpy=0. 0 0 -> xyz=0 0 0 rpy=0. 0 0.5
- joint joint2: origin xyz=0 0 -1 rpy=-0.2 0 0 -> xyz=0 0 -1 rpy=-0.5 0 0
