Commit message: Save current state.

File: src/util/pendulum.urdf (robot description, URDF)
Before this commit: robot DoublePendulum, 3 links, 2 joints
Joints:
- joint joint2: origin xyz=0 0 -1 -> xyz=0 0 -1 rpy=0 0 1.57

Commit message: URDF dynamics.

File: src/util/pendulum.urdf (robot description, URDF)
Before this commit: robot DoublePendulum, 3 links, 2 joints
Joints:
- joint joint1: origin xyz=0 1 0 -> xyz=0 1 0 rpy=0 0 1.5707963268
- joint joint2: origin xyz=0 0 -1 rpy=0 0 1.57 -> xyz=0 0 -1 rpy=0 0 1.5707963268
