Commit message: Working initital urdf parser plus examples.

File: examples/examples_files/atlas_simple.urdf (robot description, URDF)
Before this commit: robot atlas, 11 links, 10 joints
Links:
- added link head, mass 1.4199; visual mesh filename=examples/examples_files/atlas_mesh/head_chull.obj
- added link l_foot, mass 2.410; visual mesh filename=examples/examples_files/atlas_mesh/l_foot.obj; visual sphere radius=0.01
- added link l_hand, mass 0.5839
- added link l_larm, mass 3.248; visual mesh filename=examples/examples_files/atlas_mesh/r_larm.obj
- added link l_lfarm, mass 0.648; visual mesh filename=examples/examples_files/atlas_mesh/r_hand.obj
- added link l_lglut, mass 0.898; visual mesh filename=examples/examples_files/atlas_mesh/l_lglut.obj
- added link l_lleg, mass 4.515; visual mesh filename=examples/examples_files/atlas_mesh/l_lleg.obj
- added link l_talus, mass 0.125; visual mesh filename=examples/examples_files/atlas_mesh/l_talus.obj
- added link l_ufarm, mass 2.4798; visual mesh filename=examples/examples_files/atlas_mesh/r_farm.obj
- added link l_uglut, mass 1.959; visual mesh filename=examples/examples_files/atlas_mesh/l_uglut.obj
- added link l_uleg, mass 8.204; visual mesh filename=examples/examples_files/atlas_mesh/l_uleg.obj
- added link r_foot, mass 2.41; visual mesh filename=examples/examples_files/atlas_mesh/r_foot.obj; visual sphere radius=0.01
- added link r_hand, mass 0.5839
- added link r_larm, mass 3.248; visual mesh filename=examples/examples_files/atlas_mesh/r_larm.obj
- added link r_lfarm, mass 0.648; visual mesh filename=examples/examples_files/atlas_mesh/r_hand.obj
- added link r_lglut, mass 0.898; visual mesh filename=examples/examples_files/atlas_mesh/r_lglut.obj
- added link r_lleg, mass 4.515; visual mesh filename=examples/examples_files/atlas_mesh/r_lleg.obj
- added link r_talus, mass 0.125; visual mesh filename=examples/examples_files/atlas_mesh/r_talus.obj
- added link r_ufarm, mass 2.4798; visual mesh filename=examples/examples_files/atlas_mesh/r_farm.obj
- added link r_uglut, mass 1.959; visual mesh filename=examples/examples_files/atlas_mesh/r_uglut.obj
- added link r_uleg, mass 8.204; visual mesh filename=examples/examples_files/atlas_mesh/r_uleg.obj
- link l_clav: geometry visual mesh filename=examples/examples_files/atlas_mesh/r_clav.obj
- link l_scap: geometry visual mesh filename=examples/examples_files/atlas_mesh/r_scap.obj
- link l_uarm: geometry visual mesh filename=examples/examples_files/atlas_mesh/r_uarm.obj
- link ltorso: geometry visual mesh filename=examples/examples_files/atlas_mesh/ltorso.obj
- link mtorso: geometry visual mesh filename=examples/examples_files/atlas_mesh/mtorso.obj
- link pelvis: geometry visual mesh filename=examples/examples_files/atlas_mesh/pelvis.obj
- link r_clav: geometry visual mesh filename=examples/examples_files/atlas_mesh/r_clav.obj
- link r_scap: geometry visual mesh filename=examples/examples_files/atlas_mesh/r_scap.obj
- link r_uarm: geometry visual mesh filename=examples/examples_files/atlas_mesh/r_uarm.obj
- link utorso: geometry visual mesh filename=examples/examples_files/atlas_mesh/utorso.obj
Joints:
- added joint l_arm_elx: type revolute, parent l_uarm, child l_larm, origin xyz=0 -0.119 0.0092 rpy=0 0 0, axis -1.0 -0.0 -0.0, limit lower=0 upper=2.35619 effort=112 velocity=12
- added joint l_arm_lwy: type revolute, parent l_lfarm, child l_hand, origin xyz=0 0 0 rpy=0 3.14159265359 0, axis -0.0 -1.0 -0.0, limit lower=-2.9671 upper=2.9671 effort=25 velocity=10
- added joint l_arm_mwx: type revolute, parent l_ufarm, child l_lfarm, origin xyz=0 0 0 rpy=0 0 0, axis 1 0 0, limit lower=-1.7628 upper=1.7628 effort=25 velocity=10
- added joint l_arm_uwy: type revolute, parent l_larm, child l_ufarm, origin xyz=0 -0.29955 -0.00921 rpy=0 3.14159265359 0, axis -0.0 -1.0 -0.0, limit lower=-3.011 upper=3.011 effort=25 velocity=10
- added joint l_leg_akx: type revolute, parent l_talus, child l_foot, origin xyz=0 0 0 rpy=0 0 0, axis 1 0 0, limit lower=-0.8 upper=0.8 effort=360 velocity=12
- added joint l_leg_aky: type revolute, parent l_lleg, child l_talus, origin xyz=0 0 -0.422 rpy=0 0 0, axis 0 1 0, limit lower=-1 upper=0.7 effort=740 velocity=12
- added joint l_leg_hpx: type revolute, parent l_uglut, child l_lglut, origin xyz=0 0 0 rpy=0 0 0, axis 1 0 0, limit lower=-0.523599 upper=0.523599 effort=530 velocity=12
- added joint l_leg_hpy: type revolute, parent l_lglut, child l_uleg, origin xyz=0.05 0.0225 -0.066 rpy=0 0 0, axis 0 1 0, limit lower=-1.61234 upper=0.65764 effort=840 velocity=12
- added joint l_leg_hpz: type revolute, parent pelvis, child l_uglut, origin xyz=0 0.089 0 rpy=0 0 0, axis 0 0 1, limit lower=-0.174358 upper=0.786794 effort=275 velocity=12
- added joint l_leg_kny: type revolute, parent l_uleg, child l_lleg, origin xyz=-0.05 0 -0.374 rpy=0 0 0, axis 0 1 0, limit lower=0 upper=2.35637 effort=890 velocity=12
- added joint neck_ay: type revolute, parent utorso, child head, origin xyz=0.2546 0 0.6215 rpy=0 0 0, axis 0 1 0, limit lower=-0.602139 upper=1.14319 effort=25 velocity=6.28
- added joint r_arm_elx: type revolute, parent r_uarm, child r_larm, origin xyz=0 -0.119 0.0092 rpy=0 0 0, axis 1 0 0, limit lower=-2.35619 upper=0 effort=112 velocity=12
- added joint r_arm_lwy: type revolute, parent r_lfarm, child r_hand, origin xyz=0 0 0 rpy=0 0 0, axis 0 1 0, limit lower=-2.9671 upper=2.9671 effort=25 velocity=10
- added joint r_arm_mwx: type revolute, parent r_ufarm, child r_lfarm, origin xyz=0 0 0 rpy=0 0 0, axis 1 0 0, limit lower=-1.7628 upper=1.7628 effort=25 velocity=10
- added joint r_arm_uwy: type revolute, parent r_larm, child r_ufarm, origin xyz=0 -0.29955 -0.00921 rpy=0 0 0, axis 0 1 0, limit lower=-3.011 upper=3.011 effort=25 velocity=10
- added joint r_leg_akx: type revolute, parent r_talus, child r_foot, origin xyz=0 0 0 rpy=0 0 0, axis 1 0 0, limit lower=-0.8 upper=0.8 effort=360 velocity=12
- added joint r_leg_aky: type revolute, parent r_lleg, child r_talus, origin xyz=0 0 -0.422 rpy=0 0 0, axis 0 1 0, limit lower=-1 upper=0.7 effort=740 velocity=12
- added joint r_leg_hpx: type revolute, parent r_uglut, child r_lglut, origin xyz=0 0 0 rpy=0 0 0, axis 1 0 0, limit lower=-0.523599 upper=0.523599 effort=530 velocity=12
- added joint r_leg_hpy: type revolute, parent r_lglut, child r_uleg, origin xyz=0.05 -0.0225 -0.066 rpy=0 0 0, axis 0 1 0, limit lower=-1.61234 upper=0.65764 effort=840 velocity=12
- added joint r_leg_hpz: type revolute, parent pelvis, child r_uglut, origin xyz=0 -0.089 0 rpy=0 0 0, axis 0 0 1, limit lower=-0.786794 upper=0.174358 effort=275 velocity=12
- added joint r_leg_kny: type revolute, parent r_uleg, child r_lleg, origin xyz=-0.05 0 -0.374 rpy=0 0 0, axis 0 1 0, limit lower=0 upper=2.35637 effort=890 velocity=12
- joint l_arm_shz: origin xyz=0.1406 0.2256 0.4776 rpy=0 0 1.57 -> xyz=0.1406 0.2256 0.4776 rpy=0 0 3.14159265359

File: examples/examples_files/doublependulum.urdf (robot description, URDF)
Before this commit: robot DoublePendulum, 3 links, 2 joints
Links:
- link link1: geometry visual box size=.1 1 .1
Joints:
- joint joint1: origin xyz=0 1 0 rpy=0 0 1.5707963268 -> xyz=0 1 0 rpy=0.4 0 1.5707963268

Commit message: Floating base urdf.

File: examples/examples_files/atlas_simple.urdf (robot description, URDF)
Before this commit: robot atlas, 32 links, 31 joints
Links:
- removed link base_link
Joints:
- removed joint toOrigin
